File: Shield_CAN.kicad_pcb (KiCad board)
At the start: 4 copper layers, 40.1 x 27 mm, 105 parts, among them J1 Conn_01x02, J2 Conn_01x02, J3 S2B-PH-K-S_LF__SN_, J4 S2B-PH-K-S_LF__SN_, J5 Conn_01x04_Pin, J6 Conn_01x07, J8 62202821821, J9 62202821821, U1 TCAN332GDCNR, U2 STM32H563RITx, U4 LAN8742A, Y4 NX2016SA 25MHz, Y5 NX2016SA 25MHz, Y6 32.768kHz

Commit message: shield_can: swap PD2/PA6 on J9, fix PA4 on J8
The connector footprint used for J8 and J9 inverts pins 15 and 16, so
the signals assigned in the schematic did not land on the expected
physical pins of the first batch. Swap PD2 and PA6 on J9 and move PA4
accordingly on J8 so the netlist matches the actual footprint pinout,
and reroute the affected tracks on the board.
Connections:
- J8 pad 15: unconnected-(J8-Pad15) -> /PA4
- J8 pad 16: /PA4 -> unconnected-(J8-Pad16)
- J9 pad 15: /PD2 -> /PA6
- J9 pad 16: /PA6 -> /PD2
Routing:
- net /PA6: track 11.7 -> 16.3 mm
- net /PD2: track 28.6 -> 31.1 mm, vias 1 -> 2
- net /PA4: track 35.1 -> 36.1 mm
Changed lines of the file:
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@@
 			(layers "*.Cu" "*.Mask")
 			(remove_unused_layers no)
-			(net "/PD2")
+			(net "/PA6")
 			(pintype "passive")
 			(solder_mask_margin 0.102)
@@
 			(layers "*.Cu" "*.Mask")
 			(remove_unused_layers no)
-			(net "/PA6")
+			(net "/PD2")
 			(pintype "passive")
 			(solder_mask_margin 0.102)
@@
 			(layers "*.Cu" "*.Mask")
 			(remove_unused_layers no)
-			(net "unconnected-(J8-Pad15)")
-			(pintype "passive+no_connect")
+			(net "/PA4")
+			(pintype "passive")
 			(solder_mask_margin 0.102)
 		)
@@
 			(layers "*.Cu" "*.Mask")
 			(remove_unused_layers no)
-			(net "/PA4")
-			(pintype "passive")
+			(net "unconnected-(J8-Pad16)")
+			(pintype "passive+no_connect")
 			(solder_mask_margin 0.102)
 		)
@@
 	)
 	(segment
-		(start 83.7864 51.5988)
-		(end 84.4214 50.9638)
-		(width 0.15)
-		(layer "In1.Cu")
-		(net "/PA4")
-	)
-	(segment
 		(start 92.72 41.92)
 		(end 87.63 47.01)
@@
 	)
 	(segment
+		(start 83.7864 50.3288)
+		(end 84.4214 49.6938)
+		(width 0.15)
+		(layer "In1.Cu")
+		(net "/PA4")
+	)
+	(segment
 		(start 87.63 47.01)
 		(end 81.127174 47.01)
@@
 	)
 	(segment
-		(start 79.078374 51.5988)
-		(end 83.7864 51.5988)
+		(start 83.414426 51.5988)
+		(end 83.7864 51.226826)
+		(width 0.15)
+		(layer "In1.Cu")
+		(net "/PA4")
+	)
+	(segment
+		(start 83.7864 51.226826)
+		(end 83.7864 50.3288)
 		(width 0.15)
 		(layer "In1.Cu")
@@
 	)
 	(segment
+		(start 79.078374 51.5988)
+		(end 83.414426 51.5988)
+		(width 0.15)
+		(layer "In1.Cu")
+		(net "/PA4")
+	)
+	(segment
 		(start 89.22 38.68)
 		(end 89.84 39.3)
@@
 	)
 	(segment
-		(start 90.7 35.11)
-		(end 91.06 35.11)
+		(start 92.5114 27.9252)
+		(end 92.5114 27.9186)
 		(width 0.15)
 		(layer "In1.Cu")
@@
 	)
 	(segment
-		(start 92.5114 33.6586)
-		(end 92.5114 29.1952)
+		(start 90.7 35.11)
+		(end 91.15 35.11)
 		(width 0.15)
-		(layer "In1.Cu")
+		(layer "In2.Cu")
 		(net "/PA6")
 	)
 	(segment
-		(start 91.06 35.11)
-		(end 92.5114 33.6586)
+		(start 91.86 35.82)
+		(end 93.22 35.82)
 		(width 0.15)
-		(layer "In1.Cu")
+		(layer "In2.Cu")
+		(net "/PA6")
+	)
+	(segment
+		(start 93.75 34.23)
+		(end 93.1464 33.6264)
+		(width 0.15)
+		(layer "In2.Cu")
+		(net "/PA6")
+	)
+	(segment
+		(start 93.22 35.82)
+		(end 93.75 35.29)
+		(width 0.15)
+		(layer "In2.Cu")
+		(net "/PA6")
+	)
+	(segment
+		(start 93.1464 28.5602)
+		(end 92.5114 27.9252)
+		(width 0.15)
+		(layer "In2.Cu")
+		(net "/PA6")
+	)
+	(segment
+		(start 93.75 35.29)
+		(end 93.75 34.23)
+		(width 0.15)
+		(layer "In2.Cu")
+		(net "/PA6")
+	)
+	(segment
+		(start 91.15 35.11)
+		(end 91.86 35.82)
+		(width 0.15)
+		(layer "In2.Cu")
+		(net "/PA6")
+	)
+	(segment
+		(start 93.1464 33.6264)
+		(end 93.1464 28.5602)
+		(width 0.15)
+		(layer "In2.Cu")
 		(net "/PA6")
 	)
@@
 	)
 	(segment
-		(start 98.04 37.93)
-		(end 102.92 33.05)
+		(start 102.92 27.52)
+		(end 101.81 26.41)
 		(width 0.15)
 		(layer "In1.Cu")
@@
 	)
 	(segment
-		(start 102.1 26.7)
-		(end 91.1966 26.7)
+		(start 101.81 26.41)
+		(end 91.4866 26.41)
 		(width 0.15)
 		(layer "In1.Cu")
@@
 	)
 	(segment
-		(start 102.92 33.05)
-		(end 102.92 27.52)
+		(start 91.4866 26.41)
+		(end 89.9714 27.9252)
 		(width 0.15)
 		(layer "In1.Cu")
@@
 	)
 	(segment
-		(start 102.92 27.52)
-		(end 102.1 26.7)
+		(start 102.92 33.05)
+		(end 102.92 27.52)
 		(width 0.15)
 		(layer "In1.Cu")
@@
 	)
 	(segment
-		(start 91.1966 26.7)
-		(end 89.9714 27.9252)
+		(start 98.04 41.84)
+		(end 98.04 37.93)
 		(width 0.15)
 		(layer "In1.Cu")
@@
 	)
 	(segment
-		(start 98.04 41.84)
-		(end 98.04 37.93)
+		(start 98.04 37.93)
+		(end 102.92 33.05)
 		(width 0.15)
 		(layer "In1.Cu")
@@
 	)
 	(via
+		(at 93.4366 27)
+		(size 0.5)
+		(drill 0.3)
+		(layers "F.Cu" "B.Cu")
+		(net "/PD2")
+	)
+	(via
 		(at 97.02 40.71)
 		(size 0.5)
@@
 	)
 	(segment
-		(start 92.5114 27.9252)
-		(end 93.4366 27)
-		(width 0.15)
-		(layer "In1.Cu")
-		(net "/PD2")
-	)
-	(segment
-		(start 92.5114 27.9252)
-		(end 92.5114 27.9186)
-		(width 0.15)
-		(layer "In1.Cu")
-		(net "/PD2")
-	)
-	(segment
 		(start 102.53 27.73)
 		(end 102.53 32.96)
@@
 		(net "/PD2")
 	)
+	(segment
+		(start 91.8764 28.5602)
+		(end 92.5114 29.1952)
+		(width 0.15)
+		(layer "In2.Cu")
+		(net "/PD2")
+	)
+	(segment
+		(start 92.34 27)
+		(end 91.8764 27.4636)
+		(width 0.15)
+		(layer "In2.Cu")
+		(net "/PD2")
+	)
+	(segment
+		(start 91.8764 27.4636)
+		(end 91.8764 28.5602)
+		(width 0.15)
+		(layer "In2.Cu")
+		(net "/PD2")
+	)
+	(segment
+		(start 93.4366 27)
+		(end 92.34 27)
+		(width 0.15)
+		(layer "In2.Cu")
+		(net "/PD2")
+	)

Commit message: shield_can: swap D1
D1 was wired as input for Vtarget istead of an output, swap it to be able
to get a proper Vtarget when using a segger probe
Parts:
- turned D1 to 180 degrees
Connections:
- D1 pad 1: +3V3 -> Net-(D1-K)
- D1 pad 2: Net-(D1-A) -> +3V3
- J6 pad 1: Net-(D1-A) -> Net-(D1-K)
Routing:
- net Net-(D1-K): track 0.00 -> 3.29 mm, vias 0 -> 1
- net Net-(D1-A): track 3.28 -> 0.00 mm, vias 1 -> 0
Changed lines of the file:
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@@
 			(remove_unused_layers no)
 			(roundrect_rratio 0.25)
-			(net "Net-(D1-A)")
+			(net "Net-(D1-K)")
 			(pinfunction "Pin_1_1")
 			(pintype "passive")
@@
 	(footprint "Diode_SMD:D_SOD-323F"
 		(layer "B.Cu")
-		(at 103.3975 34.66)
+		(at 103.3975 34.66 180)
 		(descr "SOD-323F http://www.nxp.com/documents/outline_drawing/SOD323F.pdf")
 		(tags "SOD-323F")
@@
 		)
 		(property "Datasheet" "https://assets.nexperia.com/documents/data-sheet/BAT54J.pdf"
-			(at 0 0 180)
+			(at 0 0 0)
 			(unlocked yes)
 			(layer "B.Fab")
@@
 		)
 		(property "Description" "30V 200mA Schottky diode, SOD-323F"
-			(at 0 0 180)
+			(at 0 0 0)
 			(unlocked yes)
 			(layer "B.Fab")
@@
 		)
 		(property "Digikey_Code" "1727-4818-1-ND"
-			(at 0 0 180)
+			(at 0 0 0)
 			(unlocked yes)
 			(layer "B.Fab")
@@
 		)
 		(property "LCSC Part #" "C130415"
-			(at 0 0 180)
+			(at 0 0 0)
 			(unlocked yes)
 			(layer "B.Fab")
@@
 		)
 		(property "Mfr. Part #" "BAT54J,115 "
-			(at 0 0 180)
+			(at 0 0 0)
 			(unlocked yes)
 			(layer "B.Fab")
@@
 		(property "LCSC Part # C131394 0 0 Centrer Centrer 0 0  Mfr. Part # CC0402KRX7R9BB104 0 0 Centrer Centrer 0 0  "
 			""
-			(at 0 0 0
+			(at 0 0 180
 			)
 			(unlocked yes)
@@
 		)
 		(property "MANUFACTURER" ""
-			(at 0 0 0)
+			(at 0 0 180)
 			(unlocked yes)
 			(layer "B.Fab")
@@
 		)
 		(property "Mfr. Part # " ""
-			(at 0 0 0)
+			(at 0 0 180)
 			(unlocked yes)
 			(layer "B.Fab")
@@
 		)
 		(property "PARTREV" ""
-			(at 0 0 0)
+			(at 0 0 180)
 			(unlocked yes)
 			(layer "B.Fab")
@@
 		)
 		(property "STANDARD" ""
-			(at 0 0 0)
+			(at 0 0 180)
 			(unlocked yes)
 			(layer "B.Fab")
@@
 		)
 		(property "KLC_S3.3" ""
-			(at 0 0 0)
+			(at 0 0 180)
 			(unlocked yes)
 			(layer "B.Fab")
@@
 		)
 		(property "KLC_S4.1" ""
-			(at 0 0 0)
+			(at 0 0 180)
 			(unlocked yes)
 			(layer "B.Fab")
@@
 		(duplicate_pad_numbers_are_jumpers no)
 		(fp_line
-			(start -1.61 -0.85)
-			(end 1.05 -0.85)
+			(start -1.61 0.85)
+			(end 1.05 0.85)
 			(stroke
 				(width 0.12)
@@
 		)
 		(fp_line
-			(start -1.61 0.85)
-			(end 1.05 0.85)
+			(start -1.61 -0.85)
+			(end 1.05 -0.85)
 			(stroke
 				(width 0.12)
@@
 		)
 		(fp_line
-			(start -1.6 -0.95)
+			(start 1.6 0.95)
 			(end 1.6 -0.95)
 			(stroke
@@
 		(fp_line
 			(start -1.6 0.95)
-			(end -1.6 -0.95)
+			(end 1.6 0.95)
 			(stroke
 				(width 0.05)
@@
 		(fp_line
 			(start -1.6 0.95)
-			(end 1.6 0.95)
+			(end -1.6 -0.95)
 			(stroke
 				(width 0.05)
@@
 		)
 		(fp_line
-			(start 1.6 0.95)
+			(start -1.6 -0.95)
 			(end 1.6 -0.95)
 			(stroke
@@
 		)
 		(fp_line
-			(start -0.9 -0.7)
-			(end -0.9 0.7)
+			(start 0.9 0.7)
+			(end 0.9 -0.7)
 			(stroke
 				(width 0.1)
@@
 		)
 		(fp_line
-			(start -0.9 0.7)
-			(end 0.9 0.7)
+			(start 0.9 -0.7)
+			(end -0.9 -0.7)
 			(stroke
 				(width 0.1)
@@
 		)
 		(fp_line
-			(start -0.3 0)
-			(end -0.5 0)
+			(start 0.2 0.35)
+			(end 0.2 -0.35)
 			(stroke
 				(width 0.1)
@@
 		)
 		(fp_line
-			(start -0.3 0)
-			(end 0.2 0.35)
+			(start 0.2 0)
+			(end 0.45 0)
 			(stroke
 				(width 0.1)
@@
 		)
 		(fp_line
-			(start -0.3 0.35)
-			(end -0.3 -0.35)
+			(start 0.2 -0.35)
+			(end -0.3 0)
 			(stroke
 				(width 0.1)
@@
 		)
 		(fp_line
-			(start 0.2 -0.35)
-			(end -0.3 0)
+			(start -0.3 0.35)
+			(end -0.3 -0.35)
 			(stroke
 				(width 0.1)
@@
 		)
 		(fp_line
-			(start 0.2 0)
-			(end 0.45 0)
+			(start -0.3 0)
+			(end 0.2 0.35)
 			(stroke
 				(width 0.1)
@@
 		)
 		(fp_line
-			(start 0.2 0.35)
-			(end 0.2 -0.35)
+			(start -0.3 0)
+			(end -0.5 0)
 			(stroke
 				(width 0.1)
@@
 		)
 		(fp_line
-			(start 0.9 -0.7)
-			(end -0.9 -0.7)
+			(start -0.9 0.7)
+			(end 0.9 0.7)
 			(stroke
 				(width 0.1)
@@
 		)
 		(fp_line
-			(start 0.9 0.7)
-			(end 0.9 -0.7)
+			(start -0.9 -0.7)
+			(end -0.9 0.7)
 			(stroke
 				(width 0.1)
@@
 		)
 		(pad "1" smd roundrect
-			(at -1.1 0)
+			(at -1.1 0 180)
 			(size 0.5 0.5)
 			(layers "B.Cu" "B.Mask" "B.Paste")
 			(roundrect_rratio 0.25)
-			(net "+3V3")
+			(net "Net-(D1-K)")
 			(pinfunction "K_1")
 			(pintype "passive")
 		)
 		(pad "2" smd roundrect
-			(at 1.1 0)
+			(at 1.1 0 180)
 			(size 0.5 0.5)
 			(layers "B.Cu" "B.Mask" "B.Paste")
 			(roundrect_rratio 0.25)
-			(net "Net-(D1-A)")
+			(net "+3V3")
 			(pinfunction "A_2")
 			(pintype "passive")
@@
 	)
 	(segment
-		(start 102.2975 34.66)
-		(end 102.2975 35.5175)
-		(width 0.15)
-		(layer "B.Cu")
-		(net "+3V3")
-	)
-	(segment
 		(start 82.33 30.48)
 		(end 82.33 31.321366)
@@
 	)
 	(segment
-		(start 102.2975 35.5175)
-		(end 102.3 35.52)
-		(width 0.15)
+		(start 91.452073 43.872955)
+		(end 91.452073 44.1775)
+		(width 0.3)
 		(layer "B.Cu")
 		(net "+3V3")
 	)
 	(segment
-		(start 91.452073 43.872955)
-		(end 91.452073 44.1775)
-		(width 0.3)
+		(start 102.2975 34.66)
+		(end 102.2975 35.5175)
+		(width 0.25)
 		(layer "B.Cu")
 		(net "+3V3")
@@
 	)
 	(segment
+		(start 102.2975 35.5175)
+		(end 102.3 35.52)
+		(width 0.25)
+		(layer "B.Cu")
+		(net "+3V3")
+	)
+	(segment
 		(start 73.585 50.21)
 		(end 72.74 51.055)
@@
 	)
 	(segment
-		(start 103.44 35.635)
-		(end 103.44 34.67)
-		(width 0.15)
-		(layer "F.Cu")
-		(net "Net-(D1-A)")
-	)
-	(segment
-		(start 102.555 36.52)
-		(end 103.44 35.635)
-		(width 0.15)
-		(layer "F.Cu")
-		(net "Net-(D1-A)")
-	)
-	(via
-		(at 103.44 34.67)
-		(size 0.5)
-		(drill 0.3)
-		(layers "F.Cu" "B.Cu")
-		(net "Net-(D1-A)")
-	)
-	(segment
-		(start 103.45 34.66)
-		(end 103.44 34.67)
-		(width 0.15)
-		(layer "B.Cu")
-		(net "Net-(D1-A)")
-	)
-	(segment
-		(start 104.4975 34.66)
-		(end 103.45 34.66)
-		(width 0.15)
-		(layer "B.Cu")
-		(net "Net-(D1-A)")
-	)
-	(segment
 		(start 66.01 33.06)
 		(end 66.01 34.3375)
@@
 		(net "Net-(U1-RXD)")
 	)
+	(segment
+		(start 103.44 35.635)
+		(end 103.44 34.67)
+		(width 0.15)
+		(layer "F.Cu")
+		(net "Net-(D1-K)")
+	)
+	(segment
+		(start 102.555 36.52)
+		(end 103.44 35.635)
+		(width 0.15)
+		(layer "F.Cu")
+		(net "Net-(D1-K)")
+	)
+	(via
+		(at 103.44 34.67)
+		(size 0.5)
+		(drill 0.3)
+		(layers "F.Cu" "B.Cu")
+		(net "Net-(D1-K)")
+	)
+	(segment
+		(start 103.45 34.66)
+		(end 103.44 34.67)
+		(width 0.15)
+		(layer "B.Cu")
+		(net "Net-(D1-K)")
+	)
+	(segment
+		(start 103.44 34.67)
+		(end 104.4875 34.67)
+		(width 0.25)
+		(layer "B.Cu")
+		(net "Net-(D1-K)")
+	)
+	(segment
+		(start 104.4875 34.67)
+		(end 104.4975 34.66)
+		(width 0.25)
+		(layer "B.Cu")
+		(net "Net-(D1-K)")
+	)
 	(zone
