File: Shield_CAN.kicad_sch (KiCad schematic)
At the start: 104 parts, among them J1 Conn_01x02, J2 Conn_01x02, J3 S2B-PH-K-S_LF__SN_, J4 S2B-PH-K-S_LF__SN_, J5 Conn_01x04_Pin, J6 Conn_01x07, J8 62202821821, J9 62202821821, U1 TCAN332GDCNR, U2 STM32H563RITx, U4 LAN8742A, Y4 NX2016SA 25MHz, Y5 NX2016SA 25MHz, Y6 32.768kHz

Commit message: shield_can: swap PD2/PA6 on J9, fix PA4 on J8
The connector footprint used for J8 and J9 inverts pins 15 and 16, so
the signals assigned in the schematic did not land on the expected
physical pins of the first batch. Swap PD2 and PA6 on J9 and move PA4
accordingly on J8 so the netlist matches the actual footprint pinout,
and reroute the affected tracks on the board.
Connections:
- net PA4: now also J8.15; no longer J8.16
- net PA6: now also J9.15; no longer J9.16
- net PD2: now also J9.16; no longer J9.15

Commit message: shield_can: swap D1
D1 was wired as input for Vtarget istead of an output, swap it to be able
to get a proper Vtarget when using a segger probe
Connections:
- net +3V3: now also D1.2 (A); no longer D1.1 (K)
- net at J6.1 (Pin_1): now also D1.1 (K); no longer D1.2 (A)
Other:
- moved on the sheet: D1
